File: gmac.sch (KiCad schematic (older format))
At the start: 52 parts, among them J11 RJ45-HR911130C, U7 APX809, U8 RTL8211E, X2 25MHz

Commit message: 1.4
Fix some issues
Parts:
- J11: footprint (none) -> ~
