File: power.sch (KiCad schematic (older format))
At the start: 23 parts, among them J14 CON-1X2, J2 DC_SOCKET, U1 MP2307, U2 LM1117

Commit message: 1.4
Fix some issues
Parts:
- added C66, C72, C73: 10uF/0603, ~, symbol C
- added R76: NC/0R/1206, ~, symbol R
- C8: value 1uF/0603 -> 10uF/0603
Connections:
- wire segments 61 -> 68
Other:
- moved on the sheet: D4, R5
Changed lines of the file:
@@
 Sheet 3 11
 Title ""
-Date "19 sep 2014"
+Date "25 nov 2014"
 Rev ""
 Comp ""
@@
 L +3.3V #PWR019
 U 1 1 53DBC9E9
-P 9450 4100
-F 0 "#PWR019" H 9450 4060 30  0001 C CNN
-F 1 "+3.3V" H 9450 4210 30  0000 C CNN
-F 2 "" H 9450 4100 60  0000 C CNN
-F 3 "" H 9450 4100 60  0000 C CNN
-	1    9450 4100
+P 9450 3400
+F 0 "#PWR019" H 9450 3360 30  0001 C CNN
+F 1 "+3.3V" H 9450 3510 30  0000 C CNN
+F 2 "" H 9450 3400 60  0000 C CNN
+F 3 "" H 9450 3400 60  0000 C CNN
+	1    9450 3400
 	1    0    0    -1
 $EndComp
@@
 P 9100 4800
 F 0 "C8" H 9100 4900 40  0000 L CNN
-F 1 "1uF/0603" V 8950 4600 40  0000 L CNN
+F 1 "10uF/0603" V 8950 4600 40  0000 L CNN
 F 2 "~" H 9138 4650 30  0000 C CNN
 F 3 "~" H 9100 4800 60  0000 C CNN
@@
 L +3.3V #PWR023
 U 1 1 53DBCBAB
-P 10150 4100
-F 0 "#PWR023" H 10150 4060 30  0001 C CNN
-F 1 "+3.3V" H 10150 4210 30  0000 C CNN
-F 2 "" H 10150 4100 60  0000 C CNN
-F 3 "" H 10150 4100 60  0000 C CNN
-	1    10150 4100
+P 10850 4100
+F 0 "#PWR023" H 10850 4060 30  0001 C CNN
+F 1 "+3.3V" H 10850 4210 30  0000 C CNN
+F 2 "" H 10850 4100 60  0000 C CNN
+F 3 "" H 10850 4100 60  0000 C CNN
+	1    10850 4100
 	1    0    0    -1
 $EndComp
@@
 L R R5
 U 1 1 53DBCBC1
-P 10150 4450
-F 0 "R5" V 10230 4450 40  0000 C CNN
-F 1 "1KR/0603" V 10050 4450 40  0000 C CNN
-F 2 "~" V 10080 4450 30  0000 C CNN
-F 3 "~" H 10150 4450 30  0000 C CNN
-	1    10150 4450
+P 10850 4450
+F 0 "R5" V 10930 4450 40  0000 C CNN
+F 1 "1KR/0603" V 10750 4450 40  0000 C CNN
+F 2 "~" V 10780 4450 30  0000 C CNN
+F 3 "~" H 10850 4450 30  0000 C CNN
+	1    10850 4450
 	1    0    0    -1
 $EndComp
@@
 L LED D4
 U 1 1 53DBCBCE
-P 10150 5000
-F 0 "D4" H 10150 5100 50  0000 C CNN
-F 1 "GREEN/0603" H 10150 4900 50  0000 C CNN
-F 2 "~" H 10150 5000 60  0000 C CNN
-F 3 "~" H 10150 5000 60  0000 C CNN
-	1    10150 5000
+P 10850 5000
+F 0 "D4" H 10850 5100 50  0000 C CNN
+F 1 "GREEN/0603" H 10850 4900 50  0000 C CNN
+F 2 "~" H 10850 5000 60  0000 C CNN
+F 3 "~" H 10850 5000 60  0000 C CNN
+	1    10850 5000
 	0    1    1    0
 $EndComp
@@
 L GND #024
 U 1 1 53DBCBEA
-P 10150 5350
-F 0 "#024" H 10150 5350 30  0001 C CNN
-F 1 "GND" H 10150 5280 30  0001 C CNN
-F 2 "" H 10150 5350 60  0000 C CNN
-F 3 "" H 10150 5350 60  0000 C CNN
-	1    10150 5350
-	1    0    0    -1
-$EndComp
-Wire Wire Line
-	10150 4200 10150 4100
-Wire Wire Line
-	10150 4800 10150 4700
-Wire Wire Line
-	10150 5350 10150 5200
+P 10850 5350
+F 0 "#024" H 10850 5350 30  0001 C CNN
+F 1 "GND" H 10850 5280 30  0001 C CNN
+F 2 "" H 10850 5350 60  0000 C CNN
+F 3 "" H 10850 5350 60  0000 C CNN
+	1    10850 5350
+	1    0    0    -1
+$EndComp
+Wire Wire Line
+	10850 4200 10850 4100
+Wire Wire Line
+	10850 4800 10850 4700
+Wire Wire Line
+	10850 5350 10850 5200
 Wire Wire Line
 	9450 4600 9450 4100
@@
 Text Notes 6750 2125 0    60   ~ 0
 5V SATA POWER SUPPLY
+$Comp
+L R R76
+U 1 1 544DD81A
+P 9450 3850
+F 0 "R76" V 9530 3850 40  0000 C CNN
+F 1 "NC/0R/1206" V 9350 3850 40  0000 C CNN
+F 2 "~" V 9380 3850 30  0000 C CNN
+F 3 "~" H 9450 3850 30  0000 C CNN
+	1    9450 3850
+	-1   0    0    1
+$EndComp
+Wire Wire Line
+	9450 3600 9450 3400
+$Comp
+L +3.3V #PWR031
+U 1 1 544F8C5D
+P 9800 4100
+F 0 "#PWR031" H 9800 4060 30  0001 C CNN
+F 1 "+3.3V" H 9800 4210 30  0000 C CNN
+F 2 "" H 9800 4100 60  0000 C CNN
+F 3 "" H 9800 4100 60  0000 C CNN
+	1    9800 4100
+	1    0    0    -1
+$EndComp
+$Comp
+L C C72
+U 1 1 544F8C63
+P 9800 4450
+F 0 "C72" H 9800 4550 40  0000 L CNN
+F 1 "10uF/0603" V 9650 4250 40  0000 L CNN
+F 2 "~" H 9838 4300 30  0000 C CNN
+F 3 "~" H 9800 4450 60  0000 C CNN
+	1    9800 4450
+	1    0    0    -1
+$EndComp
+$Comp
+L GND #032
+U 1 1 544F8C6E
+P 9800 4800
+F 0 "#032" H 9800 4800 30  0001 C CNN
+F 1 "GND" H 9800 4730 30  0001 C CNN
+F 2 "" H 9800 4800 60  0000 C CNN
+F 3 "" H 9800 4800 60  0000 C CNN
+	1    9800 4800
+	1    0    0    -1
+$EndComp
+Wire Wire Line
+	9800 4250 9800 4100
+Wire Wire Line
+	9800 4650 9800 4800
+$Comp
+L +3.3V #PWR033
+U 1 1 544F8D1C
+P 10100 4100
+F 0 "#PWR033" H 10100 4060 30  0001 C CNN
+F 1 "+3.3V" H 10100 4210 30  0000 C CNN
+F 2 "" H 10100 4100 60  0000 C CNN
+F 3 "" H 10100 4100 60  0000 C CNN
+	1    10100 4100
+	1    0    0    -1
+$EndComp
+$Comp
+L C C73
+U 1 1 544F8D22
+P 10100 4450
+F 0 "C73" H 10100 4550 40  0000 L CNN
+F 1 "10uF/0603" V 9950 4250 40  0000 L CNN
+F 2 "~" H 10138 4300 30  0000 C CNN
+F 3 "~" H 10100 4450 60  0000 C CNN
+	1    10100 4450
+	1    0    0    -1
+$EndComp
+$Comp
+L GND #034
+U 1 1 544F8D28
+P 10100 4800
+F 0 "#034" H 10100 4800 30  0001 C CNN
+F 1 "GND" H 10100 4730 30  0001 C CNN
+F 2 "" H 10100 4800 60  0000 C CNN
+F 3 "" H 10100 4800 60  0000 C CNN
+	1    10100 4800
+	1    0    0    -1
+$EndComp
+Wire Wire Line
+	10100 4250 10100 4100
+Wire Wire Line
+	10100 4650 10100 4800
+$Comp
+L C C66
+U 1 1 54506B7A
+P 7850 4700
+F 0 "C66" H 7850 4800 40  0000 L CNN
+F 1 "10uF/0603" V 7700 4500 40  0000 L CNN
+F 2 "~" H 7888 4550 30  0000 C CNN
+F 3 "~" H 7850 4700 60  0000 C CNN
+	1    7850 4700
+	1    0    0    -1
+$EndComp
+$Comp
+L GND #035
+U 1 1 54506B85
+P 7850 5250
+F 0 "#035" H 7850 5250 30  0001 C CNN
+F 1 "GND" H 7850 5180 30  0001 C CNN
+F 2 "" H 7850 5250 60  0000 C CNN
+F 3 "" H 7850 5250 60  0000 C CNN
+	1    7850 5250
+	1    0    0    -1
+$EndComp
+Wire Wire Line
+	7850 4500 7850 4350
+Connection ~ 7850 4350
+Wire Wire Line
+	7850 4900 7850 5250
 $EndSCHEMATC
