File: speaker&mic.sch (KiCad schematic (older format))
At the start: 32 parts, among them J12 PJ-327F, Q3 SI2302, Q4 SI2301, Q5 SI2302, Q6 SI2301, U9 SGM358

Commit message: 1.4
Fix some issues
Parts:
- added C75, C76: 100nF/0603, ~, symbol C
- added C77, C79: 10uF/0603, ~, symbol C
- added C78: NC/10pF/0603, ~, symbol C
- added R78, R79: 22R/0603, ~, symbol R
- added R80, R81: 0R/0603, ~, symbol R
- added R82, R83: 10KR/0603, ~, symbol R
- added R84: 100R/0603, ~, symbol R
- C65: value 10uF/0603 -> 1uF/0603
Connections:
- net labels added: VMIC
- wire segments 79 -> 99
Other:
- moved on the sheet: C60, C62, C63, C65, C67, J12, R67
